File: hardware/KiCad Radio Board 2M70CM/OSS-Radio_2M70CM.kicad_sch (KiCad schematic)
At the start: 112 parts, among them J1 DF40C-24DP-0.4V, J2 P70-7000045, J3 P70-7000045, Q1 BSS138, Q2 BSS138, Q3 BSS138, U3 GRF5504, U4 TPS7A4701xRGW, U5 CC1200, U6 AT24CS01-STUM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

Commit message: more BOM changes for RF module
Parts:
- C58, C62, C63: JLCPB Part# C1852376 -> C126493; PART-NUMBER GRM1555C1H102GA1J -> GCM1555C1H102FA16D
- R10, R11, R26, R28: JLCPB Part# C5716745 -> C138022; PART-NUMBER RC0402FR-0727KP -> RC0402FR-0727KL
- R12: JLCPB Part# C4193995 -> C114756; PART-NUMBER RC0402FR-1356KL -> RC0402FR-0756KL
Changed lines of the file:
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@@
 			)
 		)
-		(property "PART-NUMBER" "GRM1555C1H102GA1J"
+		(property "PART-NUMBER" "GCM1555C1H102FA16D "
 			(at 41.91 67.31 0)
 			(effects
@@
 			)
 		)
-		(property "JLCPB Part#" "C1852376"
+		(property "JLCPB Part#" "C126493"
 			(at 41.91 67.31 90)
 			(effects
@@
 			)
 		)
-		(property "PART-NUMBER" "GRM1555C1H102GA1J"
+		(property "PART-NUMBER" "GCM1555C1H102FA16D "
 			(at 160.02 31.75 0)
 			(effects
@@
 			)
 		)
-		(property "JLCPB Part#" "C1852376"
+		(property "JLCPB Part#" "C126493"
 			(at 160.02 31.75 0)
 			(effects
@@
 			)
 		)
-		(property "PART-NUMBER" "RC0402FR-0727KP"
+		(property "PART-NUMBER" "RC0402FR-0727KL"
 			(at 161.29 166.37 0)
 			(effects
@@
 			)
 		)
-		(property "JLCPB Part#" "C5716745"
+		(property "JLCPB Part#" "C138022"
 			(at 161.29 166.37 90)
 			(effects
@@
 			)
 		)
-		(property "PART-NUMBER" "GRM1555C1H102GA1J"
+		(property "PART-NUMBER" "GCM1555C1H102FA16D "
 			(at 109.22 85.09 0)
 			(effects
@@
 			)
 		)
-		(property "JLCPB Part#" "C1852376"
+		(property "JLCPB Part#" "C126493"
 			(at 109.22 85.09 90)
 			(effects
@@
 			)
 		)
-		(property "PART-NUMBER" "RC0402FR-1356KL"
+		(property "PART-NUMBER" "RC0402FR-0756KL"
 			(at 45.72 72.39 0)
 			(effects
@@
 			)
 		)
-		(property "JLCPB Part#" "C4193995"
+		(property "JLCPB Part#" "C114756"
 			(at 45.72 72.39 90)
 			(effects
@@
 			)
 		)
-		(property "PART-NUMBER" "RC0402FR-0727KP"
+		(property "PART-NUMBER" "RC0402FR-0727KL"
 			(at 134.62 111.76 0)
 			(effects
@@
 			)
 		)
-		(property "JLCPB Part#" "C5716745"
+		(property "JLCPB Part#" "C138022"
 			(at 134.62 111.76 90)
 			(effects
@@
 			)
 		)
-		(property "PART-NUMBER" "RC0402FR-0727KP"
+		(property "PART-NUMBER" "RC0402FR-0727KL"
 			(at 166.37 152.4 0)
 			(effects
@@
 			)
 		)
-		(property "JLCPB Part#" "C5716745"
+		(property "JLCPB Part#" "C138022"
 			(at 166.37 152.4 90)
 			(effects
@@
 			)
 		)
-		(property "PART-NUMBER" "RC0402FR-0727KP"
+		(property "PART-NUMBER" "RC0402FR-0727KL"
 			(at 156.21 111.76 0)
 			(effects
@@
 			)
 		)
-		(property "JLCPB Part#" "C5716745"
+		(property "JLCPB Part#" "C138022"
 			(at 156.21 111.76 90)
 			(effects
